File: pcb/TPD.kicad_pcb (KiCad board)
At the start: 2 copper layers, 50.8 x 50.9 mm, 25 parts, among them J0 Conn_01x01, J1 Conn_01x01, J2 Conn_01x01, J3 Conn_01x01, J4 Conn_01x01, J5 Conn_01x01, J7 Conn_01x06_Pin, U1 AT42QT1070-S

Commit message: Add pin names to silkscreen
Other:
- board text added: "GND"
- board text added: "SCL"
- board text added: "SDA"
- board text added: "VCC"
- board text added: "~{CHANGE}"
- board text added: "~{RESET}"
Changed lines of the file:
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@@
     (effects (font (size 1.5 1.5) (thickness 0.3) bold) (justify left bottom mirror))
+  )
+  (gr_text "GND" (at 155.956 83.82) (layer "B.SilkS")
+    (effects (font (size 0.65 0.65) (thickness 0.12) bold) (justify mirror))
+  )
+  (gr_text "SDA" (at 154.178 81.28) (layer "B.SilkS")
+    (effects (font (size 0.65 0.65) (thickness 0.12) bold) (justify mirror))
+  )
+  (gr_text "SCL" (at 155.702 73.66) (layer "B.SilkS")
+    (effects (font (size 0.65 0.65) (thickness 0.12) bold) (justify mirror))
+  )
+  (gr_text "~{CHANGE}" (at 155.194 76.2) (layer "B.SilkS")
+    (effects (font (size 0.65 0.65) (thickness 0.12) bold) (justify mirror))
+  )
+  (gr_text "~{RESET}" (at 156.464 78.74) (layer "B.SilkS")
+    (effects (font (size 0.65 0.65) (thickness 0.12) bold) (justify mirror))
+  )
+  (gr_text "VCC" (at 154.178 86.36) (layer "B.SilkS")
+    (effects (font (size 0.65 0.65) (thickness 0.12) bold) (justify mirror))
   )
   (gr_text "Test:" (at 139.319 78.613) (layer "F.SilkS")
