File: pcb/TPD.kicad_sch (KiCad schematic)
At the start: 25 parts, among them J0 Conn_01x01, J1 Conn_01x01, J2 Conn_01x01, J3 Conn_01x01, J4 Conn_01x01, J5 Conn_01x01, J7 Conn_01x06_Pin, U1 AT42QT1070-S

Commit message: Add missing vendors
Parts:
- J7: Vendor (none) -> DigiKey; VendorId (none) -> HDR100IMP40M-G-V-SM-ND
- R1, R2, R3, R4: Vendor (none) -> HTL; VendorId (none) -> 102963
- R10, R5, R6, R7, R8, R9: Vendor (none) -> HTL; VendorId (none) -> 102967
Changed lines of the file:
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@@
+      (effects (font (size 1.27 1.27)) hide)
+    )
+    (property "Vendor" "HTL" (at 129.54 74.93 0)
+      (effects (font (size 1.27 1.27)) hide)
+    )
+    (property "VendorId" "102963" (at 129.54 74.93 0)
       (effects (font (size 1.27 1.27)) hide)
     )
@@
     )
     (property "Datasheet" "~" (at 191.77 88.9 0)
+      (effects (font (size 1.27 1.27)) hide)
+    )
+    (property "Vendor" "HTL" (at 191.77 88.9 0)
+      (effects (font (size 1.27 1.27)) hide)
+    )
+    (property "VendorId" "102967" (at 191.77 88.9 0)
       (effects (font (size 1.27 1.27)) hide)
     )
@@
       (effects (font (size 1.27 1.27)) hide)
     )
+    (property "Vendor" "HTL" (at 191.77 93.98 0)
+      (effects (font (size 1.27 1.27)) hide)
+    )
+    (property "VendorId" "102967" (at 191.77 93.98 0)
+      (effects (font (size 1.27 1.27)) hide)
+    )
     (pin "1")
     (pin "2")
@@
       (effects (font (size 1.27 1.27)) hide)
     )
+    (property "Vendor" "HTL" (at 191.77 91.44 0)
+      (effects (font (size 1.27 1.27)) hide)
+    )
+    (property "VendorId" "102967" (at 191.77 91.44 0)
+      (effects (font (size 1.27 1.27)) hide)
+    )
     (pin "1")
     (pin "2")
@@
     )
     (property "Datasheet" "~" (at 191.77 81.28 0)
+      (effects (font (size 1.27 1.27)) hide)
+    )
+    (property "Vendor" "HTL" (at 191.77 81.28 0)
+      (effects (font (size 1.27 1.27)) hide)
+    )
+    (property "VendorId" "102967" (at 191.77 81.28 0)
       (effects (font (size 1.27 1.27)) hide)
     )
@@
       (effects (font (size 1.27 1.27)) hide)
     )
+    (property "Vendor" "HTL" (at 121.92 74.93 0)
+      (effects (font (size 1.27 1.27)) hide)
+    )
+    (property "VendorId" "102963" (at 121.92 74.93 0)
+      (effects (font (size 1.27 1.27)) hide)
+    )
     (pin "1")
     (pin "2")
@@
       (effects (font (size 1.27 1.27)) hide)
     )
+    (property "Vendor" "HTL" (at 191.77 86.36 0)
+      (effects (font (size 1.27 1.27)) hide)
+    )
+    (property "VendorId" "102967" (at 191.77 86.36 0)
+      (effects (font (size 1.27 1.27)) hide)
+    )
     (pin "1")
     (pin "2")
@@
     )
     (property "Datasheet" "~" (at 191.77 83.82 0)
+      (effects (font (size 1.27 1.27)) hide)
+    )
+    (property "Vendor" "HTL" (at 191.77 83.82 0)
+      (effects (font (size 1.27 1.27)) hide)
+    )
+    (property "VendorId" "102967" (at 191.77 83.82 0)
       (effects (font (size 1.27 1.27)) hide)
     )
@@
       (effects (font (size 1.27 1.27)) hide)
     )
+    (property "Vendor" "DigiKey" (at 101.6 81.28 0)
+      (effects (font (size 1.27 1.27)) hide)
+    )
+    (property "VendorId" "HDR100IMP40M-G-V-SM-ND" (at 101.6 81.28 0)
+      (effects (font (size 1.27 1.27)) hide)
+    )
     (pin "2")
     (pin "1")
@@
       (effects (font (size 1.27 1.27)) hide)
     )
+    (property "Vendor" "HTL" (at 137.16 74.93 0)
+      (effects (font (size 1.27 1.27)) hide)
+    )
+    (property "VendorId" "102963" (at 137.16 74.93 0)
+      (effects (font (size 1.27 1.27)) hide)
+    )
     (pin "1")
     (pin "2")
@@
       (effects (font (size 1.27 1.27)) hide)
     )
+    (property "Vendor" "HTL" (at 144.78 74.93 0)
+      (effects (font (size 1.27 1.27)) hide)
+    )
+    (property "VendorId" "102963" (at 144.78 74.93 0)
+      (effects (font (size 1.27 1.27)) hide)
+    )

Commit message: Adapt vendor(id)
Parts:
- J0, J1, J2, J3, J4, J5: Vendor (none) -> -; VendorId (none) -> -
- J7: Vendor DigiKey -> HTL; VendorId HDR100IMP40M-G-V-SM-ND -> 103665
- U1: Vendor DigiKey -> HTL; VendorId AT42QT1070-SSURCT-ND -> 103664
Changed lines of the file:
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@@
+      (effects (font (size 1.27 1.27)) hide)
+    )
+    (property "Vendor" "-" (at 204.47 91.44 0)
+      (effects (font (size 1.27 1.27)) hide)
+    )
+    (property "VendorId" "-" (at 204.47 91.44 0)
       (effects (font (size 1.27 1.27)) hide)
     )
@@
       (effects (font (size 1.27 1.27)) hide)
     )
+    (property "Vendor" "-" (at 204.47 83.82 0)
+      (effects (font (size 1.27 1.27)) hide)
+    )
+    (property "VendorId" "-" (at 204.47 83.82 0)
+      (effects (font (size 1.27 1.27)) hide)
+    )
     (pin "1")
     (instances
@@
       (effects (font (size 1.27 1.27)) hide)
     )
+    (property "Vendor" "-" (at 204.47 86.36 0)
+      (effects (font (size 1.27 1.27)) hide)
+    )
+    (property "VendorId" "-" (at 204.47 86.36 0)
+      (effects (font (size 1.27 1.27)) hide)
+    )
     (pin "1")
     (instances
@@
     )
     (property "Datasheet" "~" (at 204.47 81.28 0)
+      (effects (font (size 1.27 1.27)) hide)
+    )
+    (property "Vendor" "-" (at 204.47 81.28 0)
+      (effects (font (size 1.27 1.27)) hide)
+    )
+    (property "VendorId" "-" (at 204.47 81.28 0)
       (effects (font (size 1.27 1.27)) hide)
     )
@@
       (effects (font (size 1.27 1.27)) hide)
     )
+    (property "Vendor" "-" (at 204.47 93.98 0)
+      (effects (font (size 1.27 1.27)) hide)
+    )
+    (property "VendorId" "-" (at 204.47 93.98 0)
+      (effects (font (size 1.27 1.27)) hide)
+    )
     (pin "1")
     (instances
@@
       (effects (font (size 1.27 1.27)) hide)
     )
-    (property "Vendor" "DigiKey" (at 167.64 88.9 0)
-      (effects (font (size 1.27 1.27)) hide)
-    )
-    (property "VendorId" "AT42QT1070-SSURCT-ND" (at 167.64 88.9 0)
+    (property "Vendor" "HTL" (at 167.64 88.9 0)
+      (effects (font (size 1.27 1.27)) hide)
+    )
+    (property "VendorId" "103664" (at 167.64 88.9 0)
       (effects (font (size 1.27 1.27)) hide)
     )
@@
       (effects (font (size 1.27 1.27)) hide)
     )
-    (property "Vendor" "DigiKey" (at 101.6 81.28 0)
-      (effects (font (size 1.27 1.27)) hide)
-    )
-    (property "VendorId" "HDR100IMP40M-G-V-SM-ND" (at 101.6 81.28 0)
+    (property "Vendor" "HTL" (at 101.6 81.28 0)
+      (effects (font (size 1.27 1.27)) hide)
+    )
+    (property "VendorId" "103665" (at 101.6 81.28 0)
       (effects (font (size 1.27 1.27)) hide)
     )
@@
       (effects (font (size 1.27 1.27)) hide)
     )
+    (property "Vendor" "-" (at 204.47 88.9 0)
+      (effects (font (size 1.27 1.27)) hide)
+    )
+    (property "VendorId" "-" (at 204.47 88.9 0)
+      (effects (font (size 1.27 1.27)) hide)
+    )
