File: pcb/TPD.kicad_sch (KiCad schematic)
At the start: 25 parts, among them J0 Conn_01x01, J1 Conn_01x01, J2 Conn_01x01, J3 Conn_01x01, J4 Conn_01x01, J5 Conn_01x01, J7 Conn_01x06_Pin, U1 AT42QT1070-S

Commit message: Update to KiCAD 9
Parts:
- FID1, FID2, FID3, FID4, H1, H2, J0, J1, J2, J3, J4, J5: now left out of the parts list

Commit message: Rename/Add/Remove bom fields
Parts:
- C1: HTL (none) -> 100128; Vendor HTL -> (none); VendorId 100128 -> (none)
- J0, J1, J2, J3, J4, J5: HTL (none) -> -; Vendor - -> (none); VendorId - -> (none)
- J7: HTL (none) -> 103665; Vendor HTL -> (none); VendorId 103665 -> (none)
- R1, R2, R3, R4: HTL (none) -> 102963; Vendor HTL -> (none); VendorId 102963 -> (none)
- R10, R5, R6, R7, R8, R9: HTL (none) -> 102967; Vendor HTL -> (none); VendorId 102967 -> (none)
- U1: HTL (none) -> 103664; Vendor HTL -> (none); VendorId 103664 -> (none)
